Commit message: feat(flash): compile LeRobot episodes and register RGB-D object poses
Compile spatial intervals from normal LeRobot state, action and timestamps using episode-relative indexing and both bare and .pos joint names. Add a matcher-neutral RGB-D backend that merges demo snippets in one object frame, robustly fits live correspondences, and reports explicit loss when metric evidence is insufficient.

Add the measured SO-107 gravity controller and URDF parameters from the sealed prototype as a separate LeRobot robot type. Extend the fixed-rate FLASH session with milestone-gated queue replacement and explicit receipts. Validate against the insertion recording's real dataset rows, 34 focused tests, Ruff and pre-commit.

File: src/lerobot/robots/so107_description/urdf/SO107.urdf (robot description, URDF)
Before this commit: robot SO107_urdf, 8 links, 7 joints
Links:
- link BASE_1: mass 1.4138178700759005 -> 0.1470
- link L1_1: mass 0.9302287393788501 -> 0.1000
- link L2_1: mass 1.2731856908289911 -> 0.1030
- link L3_1: mass 0.5075940741079121 -> 0.0800
- link L4_1: mass 0.6716678130372074 -> 0.0800
- link L5_1: mass 0.5075938722215222 -> 0.0790
- link L6_1: mass 0.6955792923870261 -> 0.0870
- link L7_1: mass 0.1586832108582172 -> 0.0120
Joints:
- joint S1: limit lower=-3.14159 upper=3.14159 effort=100 velocity=100 -> lower=-1.71042 upper=1.71042 effort=100 velocity=100
- joint S2: limit lower=-3.14159 upper=3.14159 effort=100 velocity=100 -> lower=-3.49066 upper=0.34907 effort=100 velocity=100
- joint S3: limit lower=-3.14159 upper=3.14159 effort=100 velocity=100 -> lower=-0.41888 upper=3.17650 effort=100 velocity=100
- joint S4: limit lower=-3.14159 upper=3.14159 effort=100 velocity=100 -> lower=-1.83260 upper=1.74533 effort=100 velocity=100
- joint S5: limit lower=-3.14159 upper=3.14159 effort=100 velocity=100 -> lower=-1.81514 upper=1.81514 effort=100 velocity=100
- joint S6: limit lower=-3.14159 upper=3.14159 effort=100 velocity=100 -> lower=-1.65806 upper=4.79966 effort=100 velocity=100
- joint S7: limit lower=-3.14159 upper=3.14159 effort=100 velocity=100 -> lower=-2.79253 upper=1.16937 effort=100 velocity=100
